File: board/main.brd (EAGLE design)
At the start: 91 x 76 mm, 53 parts, among them IC2 L6387EDIP8, IC3 L6387EDIP8, IC4 L6387EDIP8, J3 FUSE

Commit message: Added connectors to BOM
Parts:
- renumbered U$1 to J1, U$2 to J2
Changed lines of the file:
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@@
 <attribute name="VALUE" x="74" y="59.016" size="0.6096" layer="27" font="vector" ratio="20" rot="R180" align="top-center"/>
 </element>
-<element name="U$1" library="Custom_old" package="4PINVALULOK" value="HEADER4VALULOK" x="87.5" y="56" smashed="yes" rot="R90"/>
-<element name="U$2" library="Custom_old" package="6PINVALULOK" value="HEADER6" x="85" y="17" smashed="yes" rot="R90"/>
+<element name="J1" library="Custom_old" package="4PINVALULOK" value="HEADER4VALULOK" x="87.5" y="56" smashed="yes" rot="R90"/>
+<element name="J2" library="Custom_old" package="6PINVALULOK" value="HEADER6" x="85" y="17" smashed="yes" rot="R90"/>
 </elements>
 <signals>
@@
 <via x="24.4" y="7.6" extent="1-16" drill="0.6"/>
 <via x="24.4" y="4.4" extent="1-16" drill="0.6"/>
-<contactref element="U$1" pad="4"/>
-<contactref element="U$2" pad="1"/>
+<contactref element="J1" pad="4"/>
+<contactref element="J2" pad="1"/>
 </signal>
 <signal name="VDD">
@@
 <contactref element="R6" pad="P$1"/>
 <contactref element="R3" pad="P$1"/>
-<contactref element="U$2" pad="3"/>
+<contactref element="J2" pad="3"/>
 <wire x1="82" y1="34.19" x2="82" y2="31.81" width="0.254" layer="1"/>
 <wire x1="82" y1="31.81" x2="82" y2="26.5" width="0.254" layer="1"/>
@@
 <contactref element="R5" pad="P$1"/>
 <contactref element="R2" pad="P$1"/>
-<contactref element="U$2" pad="4"/>
+<contactref element="J2" pad="4"/>
 <wire x1="85" y1="34.19" x2="85" y2="31.81" width="0.254" layer="1"/>
 <wire x1="87.54" y1="14.85" x2="85.5" y2="16.89" width="0.254" layer="1"/>
@@
 <contactref element="R1" pad="P$1"/>
 <wire x1="88" y1="31.81" x2="88" y2="34.19" width="0.254" layer="1"/>
-<contactref element="U$2" pad="5"/>
+<contactref element="J2" pad="5"/>
 <wire x1="88" y1="31.81" x2="89.5" y2="30.31" width="0.254" layer="1"/>
 <wire x1="89.5" y1="13.5" x2="88.5" y2="12.5" width="0.254" layer="1"/>
@@
 <wire x1="82" y1="26.4" x2="82" y2="24.19" width="0.4064" layer="16"/>
 <wire x1="72" y1="38.8" x2="72.8" y2="38" width="0.4064" layer="1"/>
-<contactref element="U$1" pad="2"/>
-<contactref element="U$2" pad="2"/>
+<contactref element="J1" pad="2"/>
+<contactref element="J2" pad="2"/>
 <wire x1="72" y1="43.603" x2="81.897" y2="53.5" width="0.254" layer="1"/>
 <wire x1="81.897" y1="53.5" x2="86" y2="53.5" width="0.254" layer="1"/>
@@
 <signal name="N$7">
 <contactref element="R8" pad="P$1"/>
-<contactref element="U$1" pad="3"/>
+<contactref element="J1" pad="3"/>
 <wire x1="82" y1="60.2" x2="79.8" y2="58" width="0.254" layer="1"/>
 <wire x1="79.8" y1="58" x2="77.81" y2="58" width="0.254" layer="1"/>
